Commit message: Simplify OpenArm model to standalone URDF and meshes

File: robot_description/openarm_description/Openarm1.1.urdf (robot description, URDF)
Before this commit: robot OpenArm_V1.1, 22 links, 21 joints
Links:
- link base_link: geometry visual mesh filename=meshes/OpenArm_Base_1.1.STL scale=0.001 0.001 0.001
- link link_10: geometry collision mesh filename=meshes/jaw-a.STL scale=0.001 0.001 0.001; visual mesh filename=meshes/jaw-a.STL scale=0.001 0.001 0.001
- link link_11: geometry collision mesh filename=meshes/jaw-b.STL scale=0.001 0.001 0.001; visual mesh filename=meshes/jaw-b.STL scale=0.001 0.001 0.001
- link link_12: geometry collision mesh filename=meshes/J1-1.1-right.STL scale=0.001 0.001 0.001; visual mesh filename=meshes/J1-1.1-right.STL scale=0.001 0.001 0.001
- link link_13: geometry collision mesh filename=meshes/J2-1.1-right.STL scale=0.001 0.001 0.001; visual mesh filename=meshes/J2-1.1-right.STL scale=0.001 0.001 0.001
- link link_14: geometry collision mesh filename=meshes/J3-1.1-right.STL scale=0.001 0.001 0.001; visual mesh filename=meshes/J3-1.1-right.STL scale=0.001 0.001 0.001
- link link_15: geometry collision mesh filename=meshes/J4-1.1.STL scale=0.001 0.001 0.001; visual mesh filename=meshes/J4-1.1.STL scale=0.001 0.001 0.001
- link link_16: geometry collision mesh filename=meshes/J5-1.1-right.STL scale=0.001 0.001 0.001; visual mesh filename=meshes/J5-1.1-right.STL scale=0.001 0.001 0.001
- link link_17: geometry collision mesh filename=meshes/J6-1.1-right.STL scale=0.001 0.001 0.001; visual mesh filename=meshes/J6-1.1-right.STL scale=0.001 0.001 0.001
- link link_18: geometry collision mesh filename=meshes/J7-1.1-right.STL scale=0.001 0.001 0.001; visual mesh filename=meshes/J7-1.1-right.STL scale=0.001 0.001 0.001
- link link_19: geometry collision mesh filename=meshes/gripper-1.1-right.STL scale=0.001 0.001 0.001; visual mesh filename=meshes/gripper-1.1-right.STL scale=0.001 0.001 0.001
- link link_2: geometry collision mesh filename=meshes/J1-1.1.STL scale=0.001 0.001 0.001; visual mesh filename=meshes/J1-1.1.STL scale=0.001 0.001 0.001
- link link_20: geometry collision mesh filename=meshes/jaw-a.STL scale=0.001 0.001 0.001; visual mesh filename=meshes/jaw-a.STL scale=0.001 0.001 0.001
- link link_21: geometry collision mesh filename=meshes/jaw-b.STL scale=0.001 0.001 0.001; visual mesh filename=meshes/jaw-b.STL scale=0.001 0.001 0.001
- link link_3: geometry collision mesh filename=meshes/J2-1.1.STL scale=0.001 0.001 0.001; visual mesh filename=meshes/J2-1.1.STL scale=0.001 0.001 0.001
- link link_4: geometry collision mesh filename=meshes/J3-1.1.STL scale=0.001 0.001 0.001; visual mesh filename=meshes/J3-1.1.STL scale=0.001 0.001 0.001
- link link_5: geometry collision mesh filename=meshes/J4-1.1.STL scale=0.001 0.001 0.001; visual mesh filename=meshes/J4-1.1.STL scale=0.001 0.001 0.001
- link link_6: geometry collision mesh filename=meshes/J5-1.1.STL scale=0.001 0.001 0.001; visual mesh filename=meshes/J5-1.1.STL scale=0.001 0.001 0.001
- link link_7: geometry collision mesh filename=meshes/J6-1.1.STL scale=0.001 0.001 0.001; visual mesh filename=meshes/J6-1.1.STL scale=0.001 0.001 0.001
- link link_8: geometry collision mesh filename=meshes/J7-1.1.STL scale=0.001 0.001 0.001; visual mesh filename=meshes/J7-1.1.STL scale=0.001 0.001 0.001
- link link_9: geometry collision mesh filename=meshes/gripper-1.1.STL scale=0.001 0.001 0.001; visual mesh filename=meshes/gripper-1.1.STL scale=0.001 0.001 0.001
